Commit message: Drop lidar_link from the URDF to fix its double parent in TF
mapOptimization broadcasts odom -> lidar_link, but the URDF also declared
lidar_link as a fixed child of base_link, so robot_state_publisher published
base_link -> lidar_link on /tf_static. The frame ended up with two parents,
which makes tf2 lookups through it order-dependent and noisy.

The ROS 1 URDF has no lidar_link for exactly this reason - the frame is
mapOptimization's raw lidar pose, deliberately not attached to the robot
model. Neither rviz.rviz nor rviz2.rviz references it.

Co-Authored-By: Claude Opus 5 <noreply@anthropic.com>

File: config/robot.urdf.xacro (robot description, xacro)
@@ -9,10 +9,7 @@
     <origin xyz="0 0 0" rpy="0 0 0" />
   </joint>
-  <link name="lidar_link"> </link>
-  <joint name="lidar_joint" type="fixed">
-    <parent link="base_link" />
-    <child link="lidar_link" />
-    <origin xyz="0 0 0" rpy="0 0 0" />
-  </joint>
+  <!-- No lidar_link here: mapOptimization broadcasts odom -> lidar_link, so
+       declaring it in the URDF too would give the frame a second parent via
+       robot_state_publisher. Matches the ROS 1 URDF. -->
   <link name="imu_link"> </link>
   <joint name="imu_joint" type="fixed">
