Commit message: Fix curtmini frames/extrinsics, add navsat topic plumbing, document configs
params_curtmini.yaml was a copy of the ouster rig's config and did not
describe the Curt Mini at all. Corrected against the platform:

  - lidarFrame os_lidar -> os_sensor. The recorded /ouster/points are
    stamped os_lidar but the XYZ are in the sensor frame (ouster-ros
    issue #33 / PR #170: the driver's long-standing point_cloud_frame
    default was sensor_frame). Established independently of any URDF via
    IPA's base_link->xsens Rz(+90), a gyro-vs-gyro Kabsch fit between the
    bag's two IMU streams, the bag's own /tf_static, and ICP-vs-GPS
    displacement over 8/8 intervals.
  - extrinsicRot/RPY -> Rz(+90), extrinsicTrans -> mast geometry.
  - imuTopic/navsatImuTopic -> /imu/data, gpsFixTopic -> /fix.
  - Horizon_SCAN 2048 -> 1024.

fruc_curtmini.urdf.xacro: imu yaw -90 -> +90 (matches ipa320/curt_mini
sensors.xacro), os_sensor x -0.1105 -> +0.1105, os_sensor->os_lidar gets
the OS-1's real 0.0382 m + 180 deg internal transform, os_imu and gps
signs corrected.

run.launch.py: navsat_transform_node subscribes to bare 'imu' in ROS 2
where ROS 1 used 'imu/data', so a literally-ported remap matches nothing
and the GPS chain fails silently. Read navsatImuTopic/gpsFixTopic from
the params file so selecting a config selects the whole setup.

params_hesai.yaml: add broadcast_cartesian_transform_as_parent_frame.
The ROS 1 spelling is silently ignored on jazzy - navsat_transform.cpp
declares the deprecation alias with a trailing underscore.

fruc_ouster.urdf.xacro: repoint from robot_ouster_he-bo to a port of
apparatus.urdf.xacro, whose geometry reproduces FRUC ouster.yaml's
extrinsics exactly. Drop upstream's double-parented camera joint.

params_ouster.yaml and params_rslidar.yaml: adopt params_curtmini.yaml's
section headers and per-key comments. Values verified byte-identical by
parsing both revisions.

Co-Authored-By: Claude Opus 5 <noreply@anthropic.com>

File: config/fruc_curtmini.urdf.xacro (robot description, xacro)
@@ -1,28 +1,36 @@
 <?xml version="1.0"?>
-<!-- FRUC Curt Mini platform (Ouster OS-128 on a mast).
-     Ported verbatim from Forestry-Robotics-UC/fruc_lio_sam
-     launch/include/config/curtmini.urdf.xacro - geometry unchanged.
-     Use with params_ouster.yaml (lidarFrame "os_lidar"). Note the external IMU
-     is yawed -90 degrees relative to base_link; that is the physical mount, and
-     it is NOT the same thing as extrinsicRot/extrinsicRPY in the params file,
-     which describe the IMU-to-lidar rotation LIO-SAM applies internally.
+<!-- FRUC Curt Mini platform (Ouster OS-1-128 on a mast).
+     Cross-checked against the platform's description,
+     errorcodecritical/curt_dataset_recorder ros2_ws/src/curt_description/urdf/
+     {robot,sensors,properties}.xacro (their base_link_curt / imu_curt /
+     gps_curt are this file's base_link / imu / gps).
+     That repo declares os_sensor->os_lidar as IDENTITY and puts a 180 deg yaw
+     on base_link->os_sensor. Each entry is wrong on its own, but they cancel,
+     and the COMPOSITION base_link->os_lidar = Rz(180) is right.
+     Cloud +x forward and os_lidar +x backward can only both hold if the cloud
+     is not os_lidar. That is why params_curtmini.yaml sets lidarFrame to
+     os_sensor.
      Deliberately no "lidar_link": mapOptimization broadcasts odom -> lidar_link
-     itself, and declaring it here too would give that frame two parents. -->
+     itself (mapOptmization.cpp:1651) and TransformFusion broadcasts
+     odom -> base_link (imuPreintegration.cpp:149). Declaring either here would
+     give that frame two parents. -->
 <robot name="lio" xmlns:xacro="http://www.ros.org/wiki/xacro">
-  <!-- Base -->
+  <!-- Base. Its parent is odom, broadcast by TransformFusion. -->
   <link name="base_link"/>
-  <!-- External IMU -->
+  <!-- External IMU (Xsens), source of /imu/data. Yawed +90 deg on the chassis. -->
   <link name="imu"/>
   <joint name="imu_joint" type="fixed">
     <parent link="base_link"/>
     <child link="imu"/>
-    <origin xyz="0.062 0.0 0.015" rpy="0 0 -1.57079632679"/>
+    <origin xyz="0.062 0.0 0.015" rpy="0 0 1.5707963267948966"/>
   </joint>
-  <!-- Ouster sensor body -->
+  <!-- Ouster sensor body. Its +x points the way the robot drives. This is
+       also the frame the recorded point clouds are actually in, which is why
+       params_curtmini.yaml names it as lidarFrame. -->
   <link name="os_sensor"/>
   <joint name="os_sensor_joint" type="fixed">
     <parent link="base_link"/>
     <child link="os_sensor"/>
-    <origin xyz="-0.1105 0.0 0.404" rpy="0 0 0"/>
+    <origin xyz="0.1105 0.0 0.404" rpy="0 0 0"/>
   </joint>
   <!-- Ouster lidar frame -->
@@ -31,19 +39,22 @@
     <parent link="os_sensor"/>
     <child link="os_lidar"/>
-    <origin xyz="0 0 0" rpy="0 0 0"/>
+    <origin xyz="0.0 0.0 0.0382" rpy="0 0 3.141592653589793"/>
   </joint>
-  <!-- Ouster internal IMU -->
+  <!-- Ouster internal IMU. Unused by this config (only 100 Hz, and it reports
+       no orientation), kept so /ouster/imu stays resolvable. -->
   <link name="os_imu"/>
   <joint name="os_imu_joint" type="fixed">
     <parent link="os_sensor"/>
     <child link="os_imu"/>
-    <origin xyz="0 0 0" rpy="0 0 0"/>
+    <origin xyz="-0.0024 -0.0097 0.0075" rpy="0 0 0"/>
   </joint>
-  <!-- GPS -->
+  <!-- GPS antenna. The link name MUST stay "gps": navsat_transform_node looks
+       up base_link -> <frame_id of the incoming NavSatFix>, and /fix is stamped
+       "gps" in both bags. -->
   <link name="gps"/>
   <joint name="gps_joint" type="fixed">
     <parent link="base_link"/>
     <child link="gps"/>
-    <origin xyz="0.25 -0.11 0.204" rpy="0 0 0"/>
+    <origin xyz="-0.25 0.11 0.204" rpy="0 0 0"/>
   </joint>
 </robot>

File: config/fruc_ouster.urdf.xacro (robot description, xacro)
@@ -1,32 +1,110 @@
 <?xml version="1.0"?>
-<!-- FRUC Ouster OS-128 platform ("he-bo" rig).
-     Ported verbatim from Forestry-Robotics-UC/fruc_lio_sam
-     launch/include/config/robot_ouster_he-bo.urdf.xacro - geometry unchanged.
-     params_ouster.yaml sets lidarFrame to "os_lidar" and baselinkFrame to
-     "base_link"; the lidar_joint below is what makes that pair resolvable.
+<!-- FRUC Ouster OS-128 platform ("apparatus" rig).
+     Ported from Forestry-Robotics-UC/fruc_lio_sam
+     launch/include/config/apparatus.urdf.xacro - geometry unchanged.
+     NOT robot_ouster_he-bo.urdf.xacro, which this file used to transcribe.
+     That was wrong: params_ouster.yaml's extrinsics come from FRUC's
+     config/ouster.yaml, and those numbers are this rig's, exactly. Compose
+     base_link -> os_sensor -> os_lidar and invert against base_link -> xsens_imu:
+       R = Rz(180)^T                            = [-1 0 0; 0 -1 0; 0 0 1]
+       t = Rz(180)^T ((-0.015121,-0.046950,0.0586) - (0,0,0.206440))
+         = (0.015121, 0.046950, -0.147840)
+     which is ouster.yaml's extrinsicRot and extrinsicTrans [0.0151, 0.0470,
+     -0.1478] to every digit it prints. he-bo's geometry (xsens at base_link
+     identity, os_lidar at (0.15,0,0.13) unrotated) would instead demand
+     (-0.15, 0, -0.13) with R = I - nothing like it. he-bo is orphaned upstream:
+     no FRUC params file matches it, so nothing here needs it.
+     The 180 deg yaw on base_link -> os_sensor is upstream's and is kept. Note
+     it sits on the MOUNT here, unlike fruc_curtmini.urdf.xacro where the same
+     180 belongs to the OS-1's internal lidar_to_sensor_transform and sits on
+     os_sensor -> os_lidar. This file leaves os_sensor -> os_lidar identity
+     because that is how FRUC calibrated the rest of the rig against it; the
+     composition base_link -> os_lidar = Rz(180) is what the extrinsics use, and
+     it is the same either way.
+     ============================== GPS GAP ==============================
+     apparatus.urdf.xacro declares NO gps link, and params_ouster.yaml still
+     runs navsat_transform_node. That node takes gps_frame_id from the incoming
+     gps/fix header (navsat_transform.cpp:736) and does
+     lookupTransform(base_link, gps_frame_id) (:650, :697), so whatever
+     frame_id that rig's fix messages carry MUST exist below or the GPS chain
+     never initialises. No antenna position is invented here - measure it and
+     add the link. Nothing else in this file depends on it.
+     =====================================================================
      Deliberately no "lidar_link": mapOptimization broadcasts odom -> lidar_link
      itself, and declaring it here too would give that frame two parents. -->
 <robot name="lio" xmlns:xacro="http://www.ros.org/wiki/xacro">
+  <!-- Base. Upstream carries a mesh visual (apperatus.obj); dropped, the file
+       is not in the repo and robot_state_publisher does not need it. -->
   <link name="base_link"/>
-  <!-- IMU -->
+  <!-- Ouster sensor body, yawed 180 deg on the mount. -->
+  <link name="os_sensor"/>
+  <joint name="base_link_to_os_sensor" type="fixed">
+    <parent link="base_link"/>
+    <child link="os_sensor"/>
+    <origin xyz="0 0 0.206440" rpy="0 0 3.141592653589793"/>
+  </joint>
+  <!-- Ouster lidar frame. Identity to the sensor body, as upstream has it;
+       params_ouster.yaml names this as lidarFrame. -->
+  <link name="os_lidar"/>
+  <joint name="os_sensor_to_os_lidar" type="fixed">
+    <parent link="os_sensor"/>
+    <child link="os_lidar"/>
+    <origin xyz="0 0 0" rpy="0 0 0"/>
+  </joint>
+  <!-- Ouster internal IMU, from upstream's Kalibr camera-IMU calibration.
+       Unused by this config (LIO-SAM reads the Xsens), kept so /ouster/imu
+       stays resolvable. -->
+  <link name="os_imu"/>
+  <joint name="os_sensor_to_os_imu" type="fixed">
+    <parent link="os_sensor"/>
+    <child link="os_imu"/>
+    <origin xyz="-0.03516933627986119 0.026844313894637633 0.05514881960085294"
+            rpy="0.0527437133816158 -0.06297509863959863 1.5228784764076906"/>
+  </joint>
+  <!-- Xsens IMU, source of /imu/data/corrected and the frame every extrinsic
+       in params_ouster.yaml is measured against. If you change this origin,
+       recompute extrinsicTrans/extrinsicRot there.
+       robot_localization's ekf_node transforms its IMU input into
+       base_link_frame through TF, so if the /imu/data/corrected messages carry
+       a frame_id other than "xsens_imu", every IMU sample is dropped and the
+       whole GPS chain silently never initialises. LIO-SAM itself is unaffected
+       either way - it uses extrinsicRot/extrinsicRPY, not TF. -->
   <link name="xsens_imu"/>
-  <joint name="imu_joint" type="fixed">
+  <joint name="base_link_to_xsens_imu" type="fixed">
     <parent link="base_link"/>
     <child link="xsens_imu"/>
+    <origin xyz="-0.015121 -0.046950 0.0586" rpy="0 0 0"/>
+  </joint>
+  <!-- RealSense. Unused by LIO-SAM, carried over for completeness. -->
+  <link name="camera_link"/>
+  <joint name="os_sensor_to_camera_link" type="fixed">
+    <parent link="os_sensor"/>
+    <child link="camera_link"/>
+    <origin xyz="-0.018599905044461885 0.08479126746983127 -0.09082252118430068"
+            rpy="0.0013625367954899733 0.003069697768602153 1.558103710329454"/>
+  </joint>
+  <link name="camera_depth_frame"/>
+  <joint name="camera_link_to_depth_frame" type="fixed">
+    <parent link="camera_link"/>
+    <child link="camera_depth_frame"/>
     <origin xyz="0 0 0" rpy="0 0 0"/>
   </joint>
-  <!-- Ouster -->
-  <link name="os_lidar"/>
-  <joint name="lidar_joint" type="fixed">
-    <parent link="base_link"/>
-    <child link="os_lidar"/>
-    <origin xyz="0.15 0 0.13" rpy="0 0 0"/>
+  <link name="camera_depth_optical_frame"/>
+  <joint name="camera_depth_frame_to_optical" type="fixed">
+    <parent link="camera_depth_frame"/>
+    <child link="camera_depth_optical_frame"/>
+    <origin xyz="0 0 0" rpy="-1.5707963267948966 0 -1.5707963267948966"/>
   </joint>
-  <!-- GPS -->
-  <link name="gps"/>
-  <joint name="gps_joint" type="fixed">
-    <parent link="base_link"/>
-    <child link="gps"/>
-    <origin xyz="-0.20 0 0.35" rpy="0 0 0"/>
+  <link name="camera_color_frame"/>
+  <joint name="camera_link_to_color_frame" type="fixed">
+    <parent link="camera_link"/>
+    <child link="camera_color_frame"/>
+    <origin xyz="0 0 0" rpy="0 0 0"/>
+  </joint>
+  <link name="camera_color_optical_frame"/>
+  <joint name="camera_color_frame_to_optical" type="fixed">
+    <parent link="camera_color_frame"/>
+    <child link="camera_color_optical_frame"/>
+    <origin xyz="0 0 0" rpy="-1.5707963267948966 0 -1.5707963267948966"/>
   </joint>
 </robot>

Commit message: Add a Curt Mini config for 180 deg flipped clouds
The lab records custom Ouster packets and decodes them offline with their
own code. Some conversions apply a 180 deg yaw to put the points in what
curt_dataset_recorder calls "os_lidar" and some do not, so the frame is a
per-bag property that cannot be fixed once for all the existing bags.

LIO-SAM never rotates the incoming cloud - extrinsicRot/RPY/Trans apply to
the IMU only - so the whole variation is absorbed by three parameter keys
plus the frame label. params_curtmini_flipped.yaml is a copy of
params_curtmini.yaml differing in exactly those four.

fruc_curtmini.urdf.xacro gains os_sensor_flipped, a leaf at the same
origin as os_sensor yawed 180 deg. Deliberately NOT pointing lidarFrame at
os_lidar: a real OS-1 os_lidar also sits 0.0382 m above os_sensor, and the
offline decoder only rotates the points, it never translates them.

Co-Authored-By: Claude Opus 5 <noreply@anthropic.com>

File: config/fruc_curtmini.urdf.xacro (robot description, xacro)
@@ -3,12 +3,8 @@
      Cross-checked against the platform's description,
      errorcodecritical/curt_dataset_recorder ros2_ws/src/curt_description/urdf/
-     {robot,sensors,properties}.xacro (their base_link_curt / imu_curt /
-     gps_curt are this file's base_link / imu / gps).
-     That repo declares os_sensor->os_lidar as IDENTITY and puts a 180 deg yaw
-     on base_link->os_sensor. Each entry is wrong on its own, but they cancel,
-     and the COMPOSITION base_link->os_lidar = Rz(180) is right.
-     Cloud +x forward and os_lidar +x backward can only both hold if the cloud
-     is not os_lidar. That is why params_curtmini.yaml sets lidarFrame to
-     os_sensor.
+     {robot,sensors,properties}.xacro. That repo declares os_sensor->os_lidar
+     as IDENTITY and puts a 180 deg yaw on base_link->os_sensor.
+     using the stanadard: Cloud +x as forward params_curtmini.yaml sets lidarFrame
+     to os_sensor.
      Deliberately no "lidar_link": mapOptimization broadcasts odom -> lidar_link
      itself (mapOptmization.cpp:1651) and TransformFusion broadcasts
@@ -41,4 +37,15 @@
     <origin xyz="0.0 0.0 0.0382" rpy="0 0 3.141592653589793"/>
   </joint>
+  <!-- Same origin as os_sensor, yawed 180 deg. Used only by
+       params_curtmini_flipped.yaml, for bags whose offline decoder rotated the
+       points into what curt_dataset_recorder calls "os_lidar".
+       Harmless when unused: it is a leaf with one parent, and lidarFrame is
+       what selects it. -->
+  <link name="os_sensor_flipped"/>
+  <joint name="os_sensor_flipped_joint" type="fixed">
+    <parent link="os_sensor"/>
+    <child link="os_sensor_flipped"/>
+    <origin xyz="0.0 0.0 0.0" rpy="0 0 3.141592653589793"/>
+  </joint>
   <!-- Ouster internal IMU. Unused by this config (only 100 Hz, and it reports
        no orientation), kept so /ouster/imu stays resolvable. -->
@@ -51,5 +58,5 @@
   <!-- GPS antenna. The link name MUST stay "gps": navsat_transform_node looks
        up base_link -> <frame_id of the incoming NavSatFix>, and /fix is stamped
-       "gps" in both bags. -->
+       "gps" -->
   <link name="gps"/>
   <joint name="gps_joint" type="fixed">
